File: theBoerd.kicad_pcb (KiCad board)
At the start: 2 copper layers, 0 parts

Commit message: rebuild like #3 i think
Parts:
- added CH1: KS33_SW_HS, Gateron_KS33_Hotswap:Gateron-KS33-Hotswap-1U, B.Cu at (35.7, 38.1)
- added CH10: KS33_SW_HS, Gateron_KS33_Hotswap:Gateron-KS33-Hotswap-1U, B.Cu at (245.3, 38.1)
- added CH11: KS33_SW_HS, Gateron_KS33_Hotswap:Gateron-KS33-Hotswap-1U, B.Cu at (264.3, 38.1)
- added CH12: KS33_SW_HS, Gateron_KS33_Hotswap:Gateron-KS33-Hotswap-1U, B.Cu at (283.4, 38.1)
- added CH13: KS33_SW_HS, Gateron_KS33_Hotswap:Gateron-KS33-Hotswap-1U, B.Cu at (302.4, 38.1)
- added CH14: KS33_SW_HS, Gateron_KS33_Hotswap:Gateron-KS33-Hotswap-1U, B.Cu at (331.0, 38.1)
- added CH15: KS33_SW_HS, Gateron_KS33_Hotswap:Gateron-KS33-Hotswap-1U, B.Cu at (350.0, 38.1)
- added CH16: KS33_SW_HS, Gateron_KS33_Hotswap:Gateron-KS33-Hotswap-1U, B.Cu at (369.1, 38.1)
- added CH17: KS33_SW_HS, Gateron_KS33_Hotswap:Gateron-KS33-Hotswap-1U, B.Cu at (35.7, 64.3)
- added CH18: KS33_SW_HS, Gateron_KS33_Hotswap:Gateron-KS33-Hotswap-1U, B.Cu at (54.8, 64.3)
- added CH19: KS33_SW_HS, Gateron_KS33_Hotswap:Gateron-KS33-Hotswap-1U, B.Cu at (73.8, 64.3)
- added CH2: KS33_SW_HS, Gateron_KS33_Hotswap:Gateron-KS33-Hotswap-1U, B.Cu at (69.1, 38.1)
- added CH20: KS33_SW_HS, Gateron_KS33_Hotswap:Gateron-KS33-Hotswap-1U, B.Cu at (92.9, 64.3)
- added CH21: KS33_SW_HS, Gateron_KS33_Hotswap:Gateron-KS33-Hotswap-1U, B.Cu at (111.9, 64.3)
- added CH22: KS33_SW_HS, Gateron_KS33_Hotswap:Gateron-KS33-Hotswap-1U, B.Cu at (131.0, 64.3)
- added CH23: KS33_SW_HS, Gateron_KS33_Hotswap:Gateron-KS33-Hotswap-1U, B.Cu at (150.0, 64.3)
- added CH24: KS33_SW_HS, Gateron_KS33_Hotswap:Gateron-KS33-Hotswap-1U, B.Cu at (169.1, 64.3)
- added CH25: KS33_SW_HS, Gateron_KS33_Hotswap:Gateron-KS33-Hotswap-1U, B.Cu at (188.1, 64.3)
- added CH26: KS33_SW_HS, Gateron_KS33_Hotswap:Gateron-KS33-Hotswap-1U, B.Cu at (207.2, 64.3)
- added CH27: KS33_SW_HS, Gateron_KS33_Hotswap:Gateron-KS33-Hotswap-1U, B.Cu at (226.2, 64.3)
- added CH28: KS33_SW_HS, Gateron_KS33_Hotswap:Gateron-KS33-Hotswap-1U, B.Cu at (245.3, 64.3)
- added CH29: KS33_SW_HS, Gateron_KS33_Hotswap:Gateron-KS33-Hotswap-1U, B.Cu at (264.3, 64.3)
- added CH3: KS33_SW_HS, Gateron_KS33_Hotswap:Gateron-KS33-Hotswap-1U, B.Cu at (88.1, 38.1)
- added CH30: KS33_SW_HS, Gateron_KS33_Hotswap:Gateron-KS33-Hotswap-2U, B.Cu at (292.9, 64.3)
- added CH31: KS33_SW_HS, Gateron_KS33_Hotswap:Gateron-KS33-Hotswap-1.5U, B.Cu at (40.5, 83.3)
- added CH32: KS33_SW_HS, Gateron_KS33_Hotswap:Gateron-KS33-Hotswap-1U, B.Cu at (64.3, 83.3)
- added CH33: KS33_SW_HS, Gateron_KS33_Hotswap:Gateron-KS33-Hotswap-1U, B.Cu at (83.3, 83.3)
- added CH34: KS33_SW_HS, Gateron_KS33_Hotswap:Gateron-KS33-Hotswap-1U, B.Cu at (102.4, 83.3)
- added CH35: KS33_SW_HS, Gateron_KS33_Hotswap:Gateron-KS33-Hotswap-1U, B.Cu at (121.4, 83.3)
- added CH36: KS33_SW_HS, Gateron_KS33_Hotswap:Gateron-KS33-Hotswap-1U, B.Cu at (140.5, 83.3)
- added CH37: KS33_SW_HS, Gateron_KS33_Hotswap:Gateron-KS33-Hotswap-1U, B.Cu at (159.5, 83.3)
- added CH38: KS33_SW_HS, Gateron_KS33_Hotswap:Gateron-KS33-Hotswap-1U, B.Cu at (178.6, 83.3)
- added CH39: KS33_SW_HS, Gateron_KS33_Hotswap:Gateron-KS33-Hotswap-1U, B.Cu at (197.6, 83.3)
- added CH4: KS33_SW_HS, Gateron_KS33_Hotswap:Gateron-KS33-Hotswap-1U, B.Cu at (107.2, 38.1)
- added CH40: KS33_SW_HS, Gateron_KS33_Hotswap:Gateron-KS33-Hotswap-1U, B.Cu at (216.7, 83.3)
- added CH41: KS33_SW_HS, Gateron_KS33_Hotswap:Gateron-KS33-Hotswap-1U, B.Cu at (235.7, 83.3)
- added CH42: KS33_SW_HS, Gateron_KS33_Hotswap:Gateron-KS33-Hotswap-1U, B.Cu at (254.8, 83.3)
- added CH43: KS33_SW_HS, Gateron_KS33_Hotswap:Gateron-KS33-Hotswap-1U, B.Cu at (273.8, 83.3)
- added CH44: KS33_SW_HS, Gateron_KS33_Hotswap:Gateron-KS33-Hotswap-1.5U, B.Cu at (297.7, 83.3)
- added CH45: KS33_SW_HS, Gateron_KS33_Hotswap:Gateron-KS33-Hotswap-1U, B.Cu at (338.1, 83.3)
- added CH46: KS33_SW_HS, Gateron_KS33_Hotswap:Gateron-KS33-Hotswap-1U, B.Cu at (357.2, 83.3)
- added CH47: KS33_SW_HS, Gateron_KS33_Hotswap:Gateron-KS33-Hotswap-1U, B.Cu at (376.2, 83.3)
- added CH48: KS33_SW_HS, Gateron_KS33_Hotswap:Gateron-KS33-Hotswap-1.75U, B.Cu at (42.9, 102.4)
- added CH49: KS33_SW_HS, Gateron_KS33_Hotswap:Gateron-KS33-Hotswap-1U, B.Cu at (69.1, 102.4)
- added CH5: KS33_SW_HS, Gateron_KS33_Hotswap:Gateron-KS33-Hotswap-1U, B.Cu at (126.2, 38.1)
- added CH50: KS33_SW_HS, Gateron_KS33_Hotswap:Gateron-KS33-Hotswap-1U, B.Cu at (88.1, 102.4)
- added CH51: KS33_SW_HS, Gateron_KS33_Hotswap:Gateron-KS33-Hotswap-1U, B.Cu at (107.2, 102.4)
- added CH52: KS33_SW_HS, Gateron_KS33_Hotswap:Gateron-KS33-Hotswap-1U, B.Cu at (126.2, 102.4)
- added CH53: KS33_SW_HS, Gateron_KS33_Hotswap:Gateron-KS33-Hotswap-1U, B.Cu at (145.3, 102.4)
- added CH54: KS33_SW_HS, Gateron_KS33_Hotswap:Gateron-KS33-Hotswap-1U, B.Cu at (164.3, 102.4)
- added CH55: KS33_SW_HS, Gateron_KS33_Hotswap:Gateron-KS33-Hotswap-1U, B.Cu at (183.4, 102.4)
- added CH56: KS33_SW_HS, Gateron_KS33_Hotswap:Gateron-KS33-Hotswap-1U, B.Cu at (202.4, 102.4)
- added CH57: KS33_SW_HS, Gateron_KS33_Hotswap:Gateron-KS33-Hotswap-1U, B.Cu at (221.5, 102.4)
- added CH58: KS33_SW_HS, Gateron_KS33_Hotswap:Gateron-KS33-Hotswap-1U, B.Cu at (240.5, 102.4)
- added CH59: KS33_SW_HS, Gateron_KS33_Hotswap:Gateron-KS33-Hotswap-1U, B.Cu at (259.6, 102.4)
- added CH6: KS33_SW_HS, Gateron_KS33_Hotswap:Gateron-KS33-Hotswap-1U, B.Cu at (157.2, 38.1)
- added CH60: KS33_SW_HS, Gateron_KS33_Hotswap:Gateron-KS33-Hotswap-2.25U, B.Cu at (290.5, 102.4)
- added CH61: KS33_SW_HS, Gateron_KS33_Hotswap:Gateron-KS33-Hotswap-1U, B.Cu at (338.1, 102.4)
- added CH62: KS33_SW_HS, Gateron_KS33_Hotswap:Gateron-KS33-Hotswap-1U, B.Cu at (357.2, 102.4)
- added CH63: KS33_SW_HS, Gateron_KS33_Hotswap:Gateron-KS33-Hotswap-1U, B.Cu at (376.2, 102.4)
- added CH64: KS33_SW_HS, Gateron_KS33_Hotswap:Gateron-KS33-Hotswap-2.25U, B.Cu at (47.6, 121.4)
- added CH65: KS33_SW_HS, Gateron_KS33_Hotswap:Gateron-KS33-Hotswap-1U, B.Cu at (78.6, 121.4)
- added CH66: KS33_SW_HS, Gateron_KS33_Hotswap:Gateron-KS33-Hotswap-1U, B.Cu at (97.6, 121.4)
- added CH67: KS33_SW_HS, Gateron_KS33_Hotswap:Gateron-KS33-Hotswap-1U, B.Cu at (116.7, 121.4)
- added CH68: KS33_SW_HS, Gateron_KS33_Hotswap:Gateron-KS33-Hotswap-1U, B.Cu at (135.7, 121.4)
- added CH69: KS33_SW_HS, Gateron_KS33_Hotswap:Gateron-KS33-Hotswap-1U, B.Cu at (154.8, 121.4)
- added CH7: KS33_SW_HS, Gateron_KS33_Hotswap:Gateron-KS33-Hotswap-1U, B.Cu at (176.2, 38.1)
- added CH70: KS33_SW_HS, Gateron_KS33_Hotswap:Gateron-KS33-Hotswap-1U, B.Cu at (173.8, 121.4)
- added CH71: KS33_SW_HS, Gateron_KS33_Hotswap:Gateron-KS33-Hotswap-1U, B.Cu at (192.9, 121.4)
- added CH72: KS33_SW_HS, Gateron_KS33_Hotswap:Gateron-KS33-Hotswap-1U, B.Cu at (211.9, 121.4)
- added CH73: KS33_SW_HS, Gateron_KS33_Hotswap:Gateron-KS33-Hotswap-1U, B.Cu at (231.0, 121.4)
- added CH74: KS33_SW_HS, Gateron_KS33_Hotswap:Gateron-KS33-Hotswap-1U, B.Cu at (250.0, 121.4)
- added CH75: KS33_SW_HS, Gateron_KS33_Hotswap:Gateron-KS33-Hotswap-2.75U, B.Cu at (285.8, 121.4)
- added CH76: KS33_SW_HS, Gateron_KS33_Hotswap:Gateron-KS33-Hotswap-1U, B.Cu at (326.2, 121.4)
- added CH77: KS33_SW_HS, Gateron_KS33_Hotswap:Gateron-KS33-Hotswap-1U, B.Cu at (345.3, 121.4)
- added CH78: KS33_SW_HS, Gateron_KS33_Hotswap:Gateron-KS33-Hotswap-1.25U, B.Cu at (38.1, 140.5)
- added CH79: KS33_SW_HS, Gateron_KS33_Hotswap:Gateron-KS33-Hotswap-1.25U, B.Cu at (61.9, 140.5)
- added CH8: KS33_SW_HS, Gateron_KS33_Hotswap:Gateron-KS33-Hotswap-1U, B.Cu at (195.3, 38.1)
- added CH80: KS33_SW_HS, Gateron_KS33_Hotswap:Gateron-KS33-Hotswap-1.25U, B.Cu at (85.7, 140.5)
- added CH81: KS33_SW_HS, Gateron_KS33_Hotswap:Gateron-KS33-Hotswap-6.25U, B.Cu at (157.2, 140.5)
- added CH82: KS33_SW_HS, Gateron_KS33_Hotswap:Gateron-KS33-Hotswap-1.25U, B.Cu at (228.6, 140.5)
- added CH83: KS33_SW_HS, Gateron_KS33_Hotswap:Gateron-KS33-Hotswap-1.25U, B.Cu at (252.4, 140.5)
- added CH84: KS33_SW_HS, Gateron_KS33_Hotswap:Gateron-KS33-Hotswap-1.25U, B.Cu at (276.2, 140.5)
- added CH85: KS33_SW_HS, Gateron_KS33_Hotswap:Gateron-KS33-Hotswap-1.25U, B.Cu at (300.0, 140.5)
- added CH86: KS33_SW_HS, Gateron_KS33_Hotswap:Gateron-KS33-Hotswap-1U, B.Cu at (326.2, 140.5)
- added CH87: KS33_SW_HS, Gateron_KS33_Hotswap:Gateron-KS33-Hotswap-1U, B.Cu at (345.3, 140.5)
- added CH9: KS33_SW_HS, Gateron_KS33_Hotswap:Gateron-KS33-Hotswap-1U, B.Cu at (214.3, 38.1)
- added D1: D_45deg_Filled, Diode_SMD:D_1210_3225Metric, B.Cu at (42.9, 38.1)
- added D10: D_45deg_Filled, Diode_SMD:D_1210_3225Metric, B.Cu at (252.4, 38.1)
- added D11: D_45deg_Filled, Diode_SMD:D_1210_3225Metric, B.Cu at (271.5, 38.1)
- added D12: D_45deg_Filled, Diode_SMD:D_1210_3225Metric, B.Cu at (290.5, 38.1)
- added D13: D_45deg_Filled, Diode_SMD:D_1210_3225Metric, B.Cu at (309.6, 38.1)
- added D14: D_45deg_Filled, Diode_SMD:D_1210_3225Metric, B.Cu at (338.1, 38.1)
- added D15: D_45deg_Filled, Diode_SMD:D_1210_3225Metric, B.Cu at (357.2, 38.1)
- added D16: D_45deg_Filled, Diode_SMD:D_1210_3225Metric, B.Cu at (376.2, 38.1)
- added D17: D_45deg_Filled, Diode_SMD:D_1210_3225Metric, B.Cu at (42.9, 64.3)
- added D18: D_45deg_Filled, Diode_SMD:D_1210_3225Metric, B.Cu at (61.9, 64.3)
- added D19: D_45deg_Filled, Diode_SMD:D_1210_3225Metric, B.Cu at (81.0, 64.3)
- added D2: D_45deg_Filled, Diode_SMD:D_1210_3225Metric, B.Cu at (76.2, 38.1)
- added D20: D_45deg_Filled, Diode_SMD:D_1210_3225Metric, B.Cu at (100.0, 64.3)
- added D21: D_45deg_Filled, Diode_SMD:D_1210_3225Metric, B.Cu at (119.1, 64.3)
- added D22: D_45deg_Filled, Diode_SMD:D_1210_3225Metric, B.Cu at (138.1, 64.3)
- added D23: D_45deg_Filled, Diode_SMD:D_1210_3225Metric, B.Cu at (157.2, 64.3)
- added D24: D_45deg_Filled, Diode_SMD:D_1210_3225Metric, B.Cu at (176.2, 64.3)
- added D25: D_45deg_Filled, Diode_SMD:D_1210_3225Metric, B.Cu at (195.3, 64.3)
- added D26: D_45deg_Filled, Diode_SMD:D_1210_3225Metric, B.Cu at (214.3, 64.3)
- added D27: D_45deg_Filled, Diode_SMD:D_1210_3225Metric, B.Cu at (233.4, 64.3)
- added D28: D_45deg_Filled, Diode_SMD:D_1210_3225Metric, B.Cu at (252.4, 64.3)
- added D29: D_45deg_Filled, Diode_SMD:D_1210_3225Metric, B.Cu at (271.5, 64.3)
- added D3: D_45deg_Filled, Diode_SMD:D_1210_3225Metric, B.Cu at (95.2, 38.1)
- added D30: D_45deg_Filled, Diode_SMD:D_1210_3225Metric, B.Cu at (300.0, 64.3)
- added D31: D_45deg_Filled, Diode_SMD:D_1210_3225Metric, B.Cu at (47.6, 83.3)
- added D32: D_45deg_Filled, Diode_SMD:D_1210_3225Metric, B.Cu at (71.4, 83.3)
- added D33: D_45deg_Filled, Diode_SMD:D_1210_3225Metric, B.Cu at (90.5, 83.3)
- added D34: D_45deg_Filled, Diode_SMD:D_1210_3225Metric, B.Cu at (109.5, 83.3)
- added D35: D_45deg_Filled, Diode_SMD:D_1210_3225Metric, B.Cu at (128.6, 83.3)
- added D36: D_45deg_Filled, Diode_SMD:D_1210_3225Metric, B.Cu at (147.6, 83.3)
- added D37: D_45deg_Filled, Diode_SMD:D_1210_3225Metric, B.Cu at (166.7, 83.3)
- added D38: D_45deg_Filled, Diode_SMD:D_1210_3225Metric, B.Cu at (185.7, 83.3)
- added D39: D_45deg_Filled, Diode_SMD:D_1210_3225Metric, B.Cu at (204.8, 83.3)
- added D4: D_45deg_Filled, Diode_SMD:D_1210_3225Metric, B.Cu at (114.3, 38.1)
- added D40: D_45deg_Filled, Diode_SMD:D_1210_3225Metric, B.Cu at (223.8, 83.3)
- added D41: D_45deg_Filled, Diode_SMD:D_1210_3225Metric, B.Cu at (242.9, 83.3)
- added D42: D_45deg_Filled, Diode_SMD:D_1210_3225Metric, B.Cu at (261.9, 83.3)
- added D43: D_45deg_Filled, Diode_SMD:D_1210_3225Metric, B.Cu at (281.0, 83.3)
- added D44: D_45deg_Filled, Diode_SMD:D_1210_3225Metric, B.Cu at (304.8, 83.3)
- added D45: D_45deg_Filled, Diode_SMD:D_1210_3225Metric, B.Cu at (345.3, 83.3)
- added D46: D_45deg_Filled, Diode_SMD:D_1210_3225Metric, B.Cu at (364.3, 83.3)
- added D47: D_45deg_Filled, Diode_SMD:D_1210_3225Metric, B.Cu at (383.4, 83.3)
- added D48: D_45deg_Filled, Diode_SMD:D_1210_3225Metric, B.Cu at (50.0, 102.4)
- added D49: D_45deg_Filled, Diode_SMD:D_1210_3225Metric, B.Cu at (76.2, 102.4)
- added D5: D_45deg_Filled, Diode_SMD:D_1210_3225Metric, B.Cu at (133.3, 38.1)
- added D50: D_45deg_Filled, Diode_SMD:D_1210_3225Metric, B.Cu at (95.2, 102.4)
- added D51: D_45deg_Filled, Diode_SMD:D_1210_3225Metric, B.Cu at (114.3, 102.4)
- added D52: D_45deg_Filled, Diode_SMD:D_1210_3225Metric, B.Cu at (133.3, 102.4)
- added D53: D_45deg_Filled, Diode_SMD:D_1210_3225Metric, B.Cu at (152.4, 102.4)
- added D54: D_45deg_Filled, Diode_SMD:D_1210_3225Metric, B.Cu at (171.4, 102.4)
- added D55: D_45deg_Filled, Diode_SMD:D_1210_3225Metric, B.Cu at (190.5, 102.4)
- added D56: D_45deg_Filled, Diode_SMD:D_1210_3225Metric, B.Cu at (209.6, 102.4)
- added D57: D_45deg_Filled, Diode_SMD:D_1210_3225Metric, B.Cu at (228.6, 102.4)
- added D58: D_45deg_Filled, Diode_SMD:D_1210_3225Metric, B.Cu at (247.7, 102.4)
- added D59: D_45deg_Filled, Diode_SMD:D_1210_3225Metric, B.Cu at (266.7, 102.4)
- added D6: D_45deg_Filled, Diode_SMD:D_1210_3225Metric, B.Cu at (164.3, 38.1)
- added D60: D_45deg_Filled, Diode_SMD:D_1210_3225Metric, B.Cu at (297.7, 102.4)
- added D61: D_45deg_Filled, Diode_SMD:D_1210_3225Metric, B.Cu at (345.3, 102.4)
- added D62: D_45deg_Filled, Diode_SMD:D_1210_3225Metric, B.Cu at (364.3, 102.4)
- added D63: D_45deg_Filled, Diode_SMD:D_1210_3225Metric, B.Cu at (383.4, 102.4)
- added D64: D_45deg_Filled, Diode_SMD:D_1210_3225Metric, B.Cu at (54.8, 121.4)
- added D65: D_45deg_Filled, Diode_SMD:D_1210_3225Metric, B.Cu at (85.7, 121.4)
- added D66: D_45deg_Filled, Diode_SMD:D_1210_3225Metric, B.Cu at (104.8, 121.4)
- added D67: D_45deg_Filled, Diode_SMD:D_1210_3225Metric, B.Cu at (123.8, 121.4)
- added D68: D_45deg_Filled, Diode_SMD:D_1210_3225Metric, B.Cu at (142.9, 121.4)
- added D69: D_45deg_Filled, Diode_SMD:D_1210_3225Metric, B.Cu at (161.9, 121.4)
- added D7: D_45deg_Filled, Diode_SMD:D_1210_3225Metric, B.Cu at (183.4, 38.1)
- added D70: D_45deg_Filled, Diode_SMD:D_1210_3225Metric, B.Cu at (181.0, 121.4)
- added D71: D_45deg_Filled, Diode_SMD:D_1210_3225Metric, B.Cu at (200.0, 121.4)
- added D72: D_45deg_Filled, Diode_SMD:D_1210_3225Metric, B.Cu at (219.1, 121.4)
- added D73: D_45deg_Filled, Diode_SMD:D_1210_3225Metric, B.Cu at (238.1, 121.4)
- added D74: D_45deg_Filled, Diode_SMD:D_1210_3225Metric, B.Cu at (257.2, 121.4)
- added D75: D_45deg_Filled, Diode_SMD:D_1210_3225Metric, B.Cu at (292.9, 121.4)
- added D76: D_45deg_Filled, Diode_SMD:D_1210_3225Metric, B.Cu at (333.4, 121.4)
- added D77: D_45deg_Filled, Diode_SMD:D_1210_3225Metric, B.Cu at (352.4, 121.4)
- added D78: D_45deg_Filled, Diode_SMD:D_1210_3225Metric, B.Cu at (45.2, 140.5)
- added D79: D_45deg_Filled, Diode_SMD:D_1210_3225Metric, B.Cu at (69.1, 140.5)
- added D8: D_45deg_Filled, Diode_SMD:D_1210_3225Metric, B.Cu at (202.4, 38.1)
- added D80: D_45deg_Filled, Diode_SMD:D_1210_3225Metric, B.Cu at (92.9, 140.5)
- added D81: D_45deg_Filled, Diode_SMD:D_1210_3225Metric, B.Cu at (164.3, 140.5)
- added D82: D_45deg_Filled, Diode_SMD:D_1210_3225Metric, B.Cu at (235.7, 140.5)
- added D83: D_45deg_Filled, Diode_SMD:D_1210_3225Metric, B.Cu at (259.6, 140.5)
- added D84: D_45deg_Filled, Diode_SMD:D_1210_3225Metric, B.Cu at (283.4, 140.5)
- added D85: D_45deg_Filled, Diode_SMD:D_1210_3225Metric, B.Cu at (307.2, 140.5)
- added D86: D_45deg_Filled, Diode_SMD:D_1210_3225Metric, B.Cu at (333.4, 140.5)
- added D87: D_45deg_Filled, Diode_SMD:D_1210_3225Metric, B.Cu at (352.4, 140.5)
- added D9: D_45deg_Filled, Diode_SMD:D_1210_3225Metric, B.Cu at (221.5, 38.1)
- added SW1: SW_Push, Button_Switch_SMD:SW_SPDT_REED_MSDM-DT, F.Cu at (3.10, 13.4)
- added U1: BlackPill_STLINK, kicad_blackpill:BlackPill_STLINK, F.Cu at (402.4, 90.5)
- added U2: TRRS, Keebio-Parts:TRRS-PJ-320A, F.Cu at (52.4, 28.2)
Routing:
- net ROW6: track 0.00 -> 122.4 mm
- net ROW5: track 0.00 -> 77.4 mm
Other:
- board outline added: 397.7 x 131 mm
