File: theBoerdSub.kicad_pcb (KiCad board)
At the start: 2 copper layers, 173 x 120 mm, 71 parts, among them SW2 SW_Push, U1 BlackPill_STLINK, U4 TRRS

Commit message: PDF Exports
Parts:
- moved CH104 448.9 mm to (164.3, 97.6)
- moved CH108 448.9 mm to (164.3, 116.7)
- moved D102 448.9 mm to (104.8, 111.9)
- moved D106 448.9 mm to (152.4, 102.4)
- moved D109 448.9 mm to (152.4, 121.4)
- moved D111 448.9 mm to (152.6, 31.8)
- moved D112 448.9 mm to (145.6, 31.8)
- moved D113 448.9 mm to (138.6, 31.8)
- moved D91 448.9 mm to (104.8, 45.2)
- moved D95 448.9 mm to (104.8, 73.8)
- moved G*** 448.9 mm to (115.5, 32.2)
- moved CH100 448.9 mm to (59.5, 97.6)
- moved CH101 448.9 mm to (78.6, 97.6)
- moved CH105 448.9 mm to (78.6, 116.7)
- moved CH107 448.9 mm to (126.2, 97.6)
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